Commit message: fix cylinder inertia

File: urdf/commons.urdf.xacro (robot description, xacro)
@@ -22,12 +22,12 @@
   <xacro:macro name="create_box" params="m x y z *origin">
     <inertial>
-      <mass value="${m}" />
+      <mass value="${m}"/>
       <inertia
         ixx="${1/12*m*(y*y+z*z)}" ixy="0.0" ixz="0.0"
         iyy="${1/12*m*(x*x+z*z)}" iyz="0.0"
-        izz="${1/12*m*(x*x+y*y)}" />
+        izz="${1/12*m*(x*x+y*y)}"/>
     </inertial>
-    <collision>
-      <xacro:insert_block name="origin" />
+    <collision name="collision">
+      <xacro:insert_block name="origin"/>
       <geometry>
         <box size="${x} ${y} ${z}"/>
@@ -39,10 +39,10 @@
       <mass value="${m}"/>
       <inertia
-        ixx="${m*r*r}" ixy="0.0" ixz="0.0"
-        iyy="${m*r*r}" iyz="0.0"
-        izz="${m*r*r}"/>
+        ixx="${1/12*m*(3*r*r+l*l)}" ixy="0.0" ixz="0.0"
+        iyy="${1/12*m*(3*r*r+l*l)}" iyz="0.0"
+        izz="${1/2*(m*r*r)}"/>
     </inertial>
-    <collision>
-      <xacro:insert_block name="origin" />
+    <collision name="collision">
+      <xacro:insert_block name="origin"/>
       <geometry>
         <cylinder radius="${r}" length="${l}"/>
@@ -58,6 +58,6 @@
         izz="${(2/5)*m*r*r}"/>
     </inertial>
-    <collision>
-      <xacro:insert_block name="origin" />
+    <collision name="collision">
+      <xacro:insert_block name="origin"/>
       <geometry>
         <sphere radius="${r}"/>
