Commit message: set kinect_plat joint to revolute

File: urdf/actuators/torso.urdf.xacro (robot description, xacro)
@@ -94,14 +94,13 @@
       <child link="${name}"/>
     </joint>
-    <!-- should be revolute -->
-    <joint name="joint_${name}_to_${name}_sensor_plat" type="fixed">
-      <origin xyz="0.09 0 0.46" rpy="0 ${55 *(M_PI/180)} 0"/> <!-- rpy="0 0 0" -->
+    <joint name="joint_${name}_to_${name}_sensor_plat" type="revolute">
+      <origin xyz="0.09 0 0.46" rpy="0 0 0"/>
       <parent link="${name}"/>
       <child link="${name}_sensor_plat"/>
-      <!-- <axis xyz="0 1 0"/> -->
-      <!-- <limit effort="${torso_sensor_plat_effort}" velocity="${torso_sensor_plat_velocity}"
-        lower="0.0" upper="${M_PI/2}"/> -->
+      <axis xyz="0 1 0"/>
+      <limit effort="${torso_sensor_plat_effort}" velocity="${torso_sensor_plat_velocity}"
+        lower="0.0" upper="${M_PI/2}"/>
     </joint>
-    <!-- <transmission name="tran_${name}_sensor_plat">
+    <transmission name="tran_${name}_sensor_plat">
       <type>transmission_interface/SimpleTransmission</type>
       <joint name="joint_${name}_to_${name}_sensor_plat">
@@ -112,5 +111,5 @@
         <mechanicalReduction>1</mechanicalReduction>
       </actuator>
-    </transmission> -->
+    </transmission>
   </xacro:macro>
 </robot>
