Commit message: update mass

File: urdf/actuators/base.urdf.xacro (robot description, xacro)
@@ -4,9 +4,9 @@
        xmlns:interface="http://playerstage.sourceforge.net/gazebo/xmlschema/#interface"
        xmlns:xacro="http://ros.org/wiki/xacro">
-  <xacro:property name="base_mass"      value="3.00"/>
+  <xacro:property name="base_mass"      value="15.00"/>
   <xacro:property name="base_size_x"    value="0.50"/>
   <xacro:property name="base_size_y"    value="0.30"/>
   <xacro:property name="base_size_z"    value="0.07"/>
-  <xacro:property name="wheel_mass"     value="1.50"/>
+  <xacro:property name="wheel_mass"     value="2.00"/>
   <xacro:property name="wheel_radius"   value="0.10"/>
   <xacro:property name="wheel_length"   value="0.07"/>

File: urdf/actuators/torso.urdf.xacro (robot description, xacro)
@@ -4,5 +4,5 @@
        xmlns:interface="http://playerstage.sourceforge.net/gazebo/xmlschema/#interface"
        xmlns:xacro="http://ros.org/wiki/xacro">
-  <xacro:property name="big_box_mass"      value="1.00"/>
+  <xacro:property name="big_box_mass"      value="3.00"/>
   <xacro:property name="big_box_size_x"    value="0.30"/>
   <xacro:property name="big_box_size_y"    value="${base_size_y}"/>

File: urdf/sensors/asus_xtion.urdf.xacro (robot description, xacro)
@@ -1,5 +1,5 @@
 <?xml version="1.0"?>
 <robot xmlns:xacro="http://ros.org/wiki/xacro">
-  <xacro:property name="xtion_mass"   value="0.2"/>
+  <xacro:property name="xtion_mass"   value="0.10"/>
   <xacro:property name="xtion_size_x" value="0.04"/>
   <xacro:property name="xtion_size_y" value="0.18"/>

File: urdf/sensors/hokuyo_urg.urdf.xacro (robot description, xacro)
@@ -1,5 +1,5 @@
 <?xml version="1.0"?>
 <robot xmlns:xacro="http://ros.org/wiki/xacro">
-  <xacro:property name="hokuyo_urg_mass"   value="0.16"/>
+  <xacro:property name="hokuyo_urg_mass"   value="0.10"/>
   <xacro:property name="hokuyo_urg_size_x" value="0.05"/>
   <xacro:property name="hokuyo_urg_size_y" value="0.05"/>

File: urdf/sensors/hokuyo_utm.urdf.xacro (robot description, xacro)
@@ -1,5 +1,5 @@
 <?xml version="1.0"?>
 <robot xmlns:xacro="http://ros.org/wiki/xacro">
-  <xacro:property name="hokuyo_utm_mass"   value="0.270"/>
+  <xacro:property name="hokuyo_utm_mass"   value="0.10"/>
   <xacro:property name="hokuyo_utm_size_x" value="0.06"/>
   <xacro:property name="hokuyo_utm_size_y" value="0.06"/>

File: urdf/sensors/kinect_one.urdf.xacro (robot description, xacro)
@@ -1,5 +1,5 @@
 <?xml version="1.0"?>
 <robot xmlns:xacro="http://ros.org/wiki/xacro">
-  <xacro:property name="kinect_one_mass"   value="0.20"/>
+  <xacro:property name="kinect_one_mass"   value="0.10"/>
   <xacro:property name="kinect_one_size_x" value="0.07"/>
   <xacro:property name="kinect_one_size_y" value="0.28"/>

Commit message: fix wheels tfs

File: urdf/actuators/base.urdf.xacro (robot description, xacro)
@@ -4,5 +4,5 @@
        xmlns:interface="http://playerstage.sourceforge.net/gazebo/xmlschema/#interface"
        xmlns:xacro="http://ros.org/wiki/xacro">
-  <xacro:property name="base_mass"      value="15.00"/>
+  <xacro:property name="base_mass"      value="15.0"/>
   <xacro:property name="base_size_x"    value="0.50"/>
   <xacro:property name="base_size_y"    value="0.30"/>
@@ -12,15 +12,15 @@
   <xacro:property name="wheel_length"   value="0.07"/>
   <xacro:property name="wheel_gap"      value="0.02"/>
-  <xacro:property name="wheel_effort"   value="30" />
-  <xacro:property name="whell_velocity" value="0.5" />
+  <xacro:property name="wheel_effort"   value="30.0" />
+  <xacro:property name="wheel_velocity" value="0.50" />
   <xacro:macro name="wheel" params="name parent *origin *visual">
     <link name="${name}">
       <xacro:create_cylinder m="${wheel_mass}" r="${wheel_radius}" l="${wheel_length}">
-        <origin xyz="0 0 0" rpy="0 0 0"/>
+        <origin xyz="0 0 0" rpy="${M_PI/2} 0 0"/>
       </xacro:create_cylinder>
       <xacro:insert_block name="visual"/>
       <!-- wheel suport: used to reduce wheel contact in the floor -->
       <xacro:create_sphere m="${0.001}" r="${0.005}">
-        <origin xyz="0 -${wheel_radius} 0" rpy="0 0 0"/>
+        <origin xyz="0 0 -${wheel_radius}" rpy="0 0 0"/>
       </xacro:create_sphere>
       <!-- wheel suport -->
@@ -32,18 +32,7 @@
       <child link="${name}"/>
       <!-- enable when joint type is continuous -->
-      <!-- <axis xyz="0 0 1"/>  -->
+      <!-- <axis xyz="0 1 0"/> -->
       <!-- <limit effort="${wheel_effort}" velocity="${wheel_velocity}"/> -->
     </joint>
-    <!-- wheel suport: used to reduce wheel contact in the floor -->
-    <!-- <link name="${name}_support">
-      <xacro:create_sphere m="${0.001}" r="${0.005}">
-        <origin xyz="0 0 0" rpy="0 0 0"/>
-      </xacro:create_sphere>
-    </link>
-    <joint name="joint_${name}_to_${name}_support" type="fixed">
-      <origin xyz="0 -${wheel_radius} 0" rpy="0 0 0"/>
-      <parent link="${name}"/>
-      <child link="${name}_support"/>
-    </joint> -->
   </xacro:macro>
   <xacro:macro name="base" params="name">
@@ -71,7 +60,7 @@
       <origin
         xyz="${0.4*base_size_x} -${base_size_y/2+wheel_length/2+wheel_gap} 0.0"
-        rpy="${M_PI/2} 0 0" />
+        rpy="0 0 0" />
       <visual>
-        <origin xyz="0 0 0.045" rpy="0 -${M_PI/2} 0"/>
+        <origin xyz="0 -0.045 0" rpy=" 0 0 -${M_PI/2}"/>
         <material name="white"/>
         <geometry>
@@ -84,7 +73,7 @@
       <origin
         xyz="${0.4*base_size_x} ${base_size_y/2+wheel_length/2+wheel_gap} 0.0"
-        rpy="${M_PI/2} 0 0" />
+        rpy="0 0 0" />
       <visual>
-        <origin xyz="0 0 -0.045" rpy="0 ${M_PI/2} 0"/>
+        <origin xyz="0 0.045 0" rpy=" 0 0 ${M_PI/2}"/>
         <material name="white"/>
         <geometry>
@@ -97,7 +86,7 @@
       <origin
         xyz="-${0.4*base_size_x} -${base_size_y/2+wheel_length/2+wheel_gap} 0.0"
-        rpy="${M_PI/2} 0 0"/>
+        rpy="0 0 0"/>
       <visual>
-        <origin xyz="0 0 0.045" rpy="0 -${M_PI/2} 0"/>
+        <origin xyz="0 -0.045 0" rpy="0 0 -${M_PI/2}"/>
         <material name="white"/>
         <geometry>
@@ -110,7 +99,7 @@
       <origin
         xyz="-${0.4*base_size_x} ${base_size_y/2+wheel_length/2+wheel_gap} 0.0"
-        rpy="${M_PI/2} 0 0"/>
+        rpy="0 0 0"/>
       <visual>
-        <origin xyz="0 0 -0.045" rpy="0 ${M_PI/2} 0"/>
+        <origin xyz="0 0.045 0" rpy="0 0 ${M_PI/2}"/>
         <material name="white"/>
         <geometry>

Commit message: update

File: urdf/actuators/base.urdf.xacro (robot description, xacro)
@@ -4,5 +4,5 @@
        xmlns:interface="http://playerstage.sourceforge.net/gazebo/xmlschema/#interface"
        xmlns:xacro="http://ros.org/wiki/xacro">
-  <xacro:property name="base_mass"      value="20.0"/>
+  <xacro:property name="base_mass"      value="99.0"/>
   <xacro:property name="base_size_x"    value="0.50"/>
   <xacro:property name="base_size_y"    value="0.30"/>

File: urdf/actuators/head.urdf.xacro (robot description, xacro)
@@ -58,5 +58,6 @@
       <parent link="${parent}"/>
       <axis xyz="0 0 1"/>
-      <limit effort="${head_effort}" velocity="${head_velocity}" lower="-${M_PI/2}" upper="${M_PI/2}"/>
+      <limit effort="${head_effort}" velocity="${head_velocity}"
+        lower="${-M_PI/2}" upper="${M_PI/2}"/>
     </joint>
     <transmission name="tran_${name}">

File: urdf/sensors/kinect_one.urdf.xacro (robot description, xacro)
@@ -28,5 +28,5 @@
     </joint>
     <link name="${name}_depth"/>
-    <joint name="$joint_${name}_to_${name}_depth" type="fixed">
+    <joint name="joint_${name}_to_${name}_depth" type="fixed">
       <origin xyz="0.0 -0.049 0.0" rpy="0 0 0" />
       <parent link="${name}" />
