Commit message: update sensors config and robot mass distribution,

File: robots/hera_full.urdf.xacro (robot description, xacro)
@@ -75,5 +75,5 @@
   <xacro:gazebo_hokuyo_utm
     reference="base_scan_front"
-    update_rate="10"
+    update_rate="30"
     min_angle="-1.45"
     max_angle="1.45"/>
@@ -81,5 +81,5 @@
   <xacro:gazebo_hokuyo_urg
     reference="base_scan_back"
-    update_rate="10"
+    update_rate="30"
     min_angle="-1.45"
     max_angle="1.45" />
@@ -87,8 +87,8 @@
   <xacro:gazebo_xtion
     reference="xtion"
-    update_rate="10"/>
+    update_rate="30"/>
   <!-- kinect_one -->
   <xacro:gazebo_kinect_one
     reference="kinect_one"
-    update_rate="10"/>
+    update_rate="30"/>
 </robot>

File: urdf/actuators/base.urdf.xacro (robot description, xacro)
@@ -4,9 +4,9 @@
        xmlns:interface="http://playerstage.sourceforge.net/gazebo/xmlschema/#interface"
        xmlns:xacro="http://ros.org/wiki/xacro">
-  <xacro:property name="base_mass"      value="15.0"/>
+  <xacro:property name="base_mass"      value="20.0"/>
   <xacro:property name="base_size_x"    value="0.50"/>
   <xacro:property name="base_size_y"    value="0.30"/>
   <xacro:property name="base_size_z"    value="0.07"/>
-  <xacro:property name="wheel_mass"     value="2.00"/>
+  <xacro:property name="wheel_mass"     value="2.50"/>
   <xacro:property name="wheel_radius"   value="0.10"/>
   <xacro:property name="wheel_length"   value="0.07"/>

File: urdf/actuators/torso.urdf.xacro (robot description, xacro)
@@ -4,5 +4,5 @@
        xmlns:interface="http://playerstage.sourceforge.net/gazebo/xmlschema/#interface"
        xmlns:xacro="http://ros.org/wiki/xacro">
-  <xacro:property name="big_box_mass"      value="3.00"/>
+  <xacro:property name="big_box_mass"      value="1.00"/>
   <xacro:property name="big_box_size_x"    value="0.30"/>
   <xacro:property name="big_box_size_y"    value="${base_size_y}"/>
@@ -94,13 +94,14 @@
       <child link="${name}"/>
     </joint>
-    <joint name="joint_${name}_to_${name}_sensor_plat" type="revolute">
-      <origin xyz="0.09 0 0.46" rpy="0 0 0"/>
+    <!-- should be revolute -->
+    <joint name="joint_${name}_to_${name}_sensor_plat" type="fixed">
+      <origin xyz="0.09 0 0.46" rpy="0 ${55 *(M_PI/180)} 0"/> <!-- rpy="0 0 0" -->
       <parent link="${name}"/>
       <child link="${name}_sensor_plat"/>
-      <axis xyz="0 1 0"/>
-      <limit effort="${torso_sensor_plat_effort}" velocity="${torso_sensor_plat_velocity}"
-        lower="0.0" upper="${M_PI/2}"/>
+      <!-- <axis xyz="0 1 0"/> -->
+      <!-- <limit effort="${torso_sensor_plat_effort}" velocity="${torso_sensor_plat_velocity}"
+        lower="0.0" upper="${M_PI/2}"/> -->
     </joint>
-    <transmission name="tran_${name}_sensor_plat">
+    <!-- <transmission name="tran_${name}_sensor_plat">
       <type>transmission_interface/SimpleTransmission</type>
       <joint name="joint_${name}_to_${name}_sensor_plat">
@@ -111,5 +112,5 @@
         <mechanicalReduction>1</mechanicalReduction>
       </actuator>
-    </transmission>
+    </transmission> -->
   </xacro:macro>
 </robot>

File: urdf/sensors/asus_xtion.urdf.xacro (robot description, xacro)
@@ -1,5 +1,5 @@
 <?xml version="1.0"?>
 <robot xmlns:xacro="http://ros.org/wiki/xacro">
-  <xacro:property name="xtion_mass"   value="0.10"/>
+  <xacro:property name="xtion_mass"   value="0.01"/>
   <xacro:property name="xtion_size_x" value="0.04"/>
   <xacro:property name="xtion_size_y" value="0.18"/>

File: urdf/sensors/hokuyo_urg.urdf.xacro (robot description, xacro)
@@ -1,5 +1,5 @@
 <?xml version="1.0"?>
 <robot xmlns:xacro="http://ros.org/wiki/xacro">
-  <xacro:property name="hokuyo_urg_mass"   value="0.10"/>
+  <xacro:property name="hokuyo_urg_mass"   value="0.01"/>
   <xacro:property name="hokuyo_urg_size_x" value="0.05"/>
   <xacro:property name="hokuyo_urg_size_y" value="0.05"/>

File: urdf/sensors/hokuyo_utm.urdf.xacro (robot description, xacro)
@@ -1,5 +1,5 @@
 <?xml version="1.0"?>
 <robot xmlns:xacro="http://ros.org/wiki/xacro">
-  <xacro:property name="hokuyo_utm_mass"   value="0.10"/>
+  <xacro:property name="hokuyo_utm_mass"   value="0.01"/>
   <xacro:property name="hokuyo_utm_size_x" value="0.06"/>
   <xacro:property name="hokuyo_utm_size_y" value="0.06"/>

File: urdf/sensors/kinect_one.urdf.xacro (robot description, xacro)
@@ -1,5 +1,5 @@
 <?xml version="1.0"?>
 <robot xmlns:xacro="http://ros.org/wiki/xacro">
-  <xacro:property name="kinect_one_mass"   value="0.10"/>
+  <xacro:property name="kinect_one_mass"   value="0.01"/>
   <xacro:property name="kinect_one_size_x" value="0.07"/>
   <xacro:property name="kinect_one_size_y" value="0.28"/>

File: urdf/simulation/asus_xtion.gazebo.xacro (robot description, xacro)
@@ -10,10 +10,10 @@
             <image>
               <format>R8G8B8</format>
-              <width>640</width>
-              <height>480</height>
+              <width>${640/20}</width>
+              <height>${480/20}</height>
             </image>
             <clip>
-              <near>0.5</near>
-              <far>10</far>
+              <near>0.8</near>
+              <far>3.5</far>
             </clip>
           </camera>

File: urdf/simulation/kinect_one.gazebo.xacro (robot description, xacro)
@@ -10,9 +10,9 @@
                 <image>
                   <format>R8G8B8</format>
-                  <width>640</width>
-                  <height>480</height>
+                  <width>${640/20}</width>
+                  <height>${480/20}</height>
                 </image>
                 <clip>
-                    <near>0.5</near>
+                    <near>0.4</near>
                     <far>10</far>
                 </clip>

Commit message: add manipulator

File: robots/hera_full.urdf.xacro (robot description, xacro)
@@ -15,4 +15,5 @@
   <xacro:include filename="$(find hera_description)/urdf/actuators/torso.urdf.xacro" />
   <xacro:include filename="$(find hera_description)/urdf/actuators/head.urdf.xacro" />
+  <xacro:include filename="$(find hera_description)/urdf/actuators/manipulator/manip.urdf.xacro" />
   <!-- sensors -->
   <xacro:include filename="$(find hera_description)/urdf/sensors/hokuyo_utm.urdf.xacro"/>
@@ -22,5 +23,4 @@
   <!-- simulation -->
   <xacro:include filename="$(find hera_description)/urdf/simulation/colors.gazebo.xacro" />
-  <xacro:include filename="$(find hera_description)/urdf/simulation/control.gazebo.xacro" />
   <xacro:include filename="$(find hera_description)/urdf/simulation/base.gazebo.xacro"/>
   <xacro:include filename="$(find hera_description)/urdf/simulation/hokuyo_utm.gazebo.xacro" />
@@ -28,4 +28,5 @@
   <xacro:include filename="$(find hera_description)/urdf/simulation/asus_xtion.gazebo.xacro" />
   <xacro:include filename="$(find hera_description)/urdf/simulation/kinect_one.gazebo.xacro" />
+  <xacro:include filename="$(find hera_description)/urdf/simulation/manipulator.gazebo.xacro" />
 <!-- ####################################################################### -->
 <!-- ######################## robot parts ################################## -->
@@ -66,4 +67,12 @@
     <origin xyz="0.05 0 0.1" rpy="0 0 0" />
   </xacro:kinect_one>
+  <!--torso suporte-->
+  <xacro:create_manip_support_link
+    parent="torso"/>
+  <!--torso backrest-->
+  <xacro:create_backrest_link
+    parent="torso"/>
+  <!-- manip -->
+  <xacro:manipulator/>
 <!-- ####################################################################### -->
 <!-- ####################### gazebo extensions ##############################-->
@@ -92,3 +101,4 @@
     reference="kinect_one"
     update_rate="30"/>
+  <xacro:manip_transmission/>
 </robot>

File: urdf/actuators/torso.urdf.xacro (robot description, xacro)
@@ -71,4 +71,11 @@
         </geometry>
       </visual>
+      <collision>
+        <origin xyz="0 0 -0.5" rpy="0 0 0"/>
+        <material name="dark_grey"/>
+        <geometry>
+          <mesh filename="package://hera_description/meshes/torso.stl"/>
+        </geometry>
+      </collision>
     </link>
     <!-- sensor plat -->
@@ -113,3 +120,61 @@
     </transmission>
   </xacro:macro>
+  <!--manip_support_link-->
+  <xacro:macro name="create_manip_support_link" params="parent">
+    <link name="manip_support_link">
+      <visual>
+        <origin xyz="0 0 0" rpy="0 0 0" />
+        <geometry>
+          <mesh filename="package://hera_description/meshes/manip_meshes/manip_support.STL"/>
+        </geometry>
+        <material name="grey">
+          <color rgba="0.792156862745098 0.819607843137255 0.933333333333333 1" />
+        </material>
+      </visual>
+      <collision>
+        <origin xyz="0 0 0" rpy="0 0 0" />
+        <geometry>
+          <mesh filename="package://hera_description/meshes/manip_meshes/manip_support.STL"/>
+        </geometry>
+      </collision>
+      <xacro:inertial_manip_support_link mass="0.659217140679788"/>
+    </link>
+    <!--manip_support_joint-->
+    <joint name="manip_support_joint" type="fixed">
+      <origin xyz="0.04525 0 0.0285" rpy="0 0 0" />
+      <parent link="${parent}" />
+      <child link="manip_support_link" />
+      <axis xyz="0 0 0" />
+      <limit lower="0" upper="0" effort="0" velocity="0" />
+    </joint>
+  </xacro:macro>
+  <!--backrest_link-->
+  <xacro:macro name="create_backrest_link" params="parent">
+    <link name="backrest_link">
+      <visual>
+        <origin xyz="0 0 0" rpy="0 0 0" />
+        <geometry>
+          <mesh filename="package://hera_description/meshes/manip_meshes/backrest.STL"/>
+        </geometry>
+        <material name="grey">
+          <color rgba="0.898039215686275 0.917647058823529 0.929411764705882 1" />
+        </material>
+      </visual>
+      <collision>
+        <origin xyz="0 0 0" rpy="0 0 0" />
+        <geometry>
+          <mesh filename="package://hera_description/meshes/manip_meshes/backrest.STL"/>
+        </geometry>
+      </collision>
+      <xacro:inertial_backrest_link mass="0.0709912944888601"/>
+    </link>
+    <!--backrest_joint-->
+    <joint name="backrest_joint" type="fixed">
+      <origin xyz="0.028 0.0066709 0.053" rpy="0 0 0" />
+      <parent link="${parent}" />
+      <child link="backrest_link" />
+      <axis xyz="0 0 0" />
+      <limit effort="0" velocity="0" />
+    </joint>
+  </xacro:macro>
 </robot>

File: urdf/simulation/kinect_one.gazebo.xacro (robot description, xacro)
@@ -10,6 +10,6 @@
                 <image>
                   <format>R8G8B8</format>
-                  <width>${640/20}</width>
-                  <height>${480/20}</height>
+                  <width>${640}</width>
+                  <height>${480}</height>
                 </image>
                 <clip>

Commit message: update urdf

File: robots/hera_full.urdf.xacro (robot description, xacro)
@@ -29,4 +29,5 @@
   <xacro:include filename="$(find hera_description)/urdf/simulation/kinect_one.gazebo.xacro" />
   <xacro:include filename="$(find hera_description)/urdf/simulation/manipulator.gazebo.xacro" />
+  <xacro:include filename="$(find hera_description)/urdf/simulation/control.gazebo.xacro" />
 <!-- ####################################################################### -->
 <!-- ######################## robot parts ################################## -->
@@ -80,5 +81,6 @@
   <!-- base -->
   <xacro:gazebo_base
-    reference="base"/>
+    reference="base"
+    update_rate="30"/>
   <!-- hokuyo_utm -->
   <xacro:gazebo_hokuyo_utm

File: urdf/actuators/manipulator/simulation_gripper/robotiq_85_gripper.xacro (robot description, xacro)
@@ -2,9 +2,9 @@
 <robot name="robotiq_85_gripper" xmlns:xacro="http://www.ros.org/wiki/xacro">
   <xacro:include filename="$(find robotiq_description)/urdf/robotiq_85_gripper.urdf.xacro" />
-  <gazebo>
+  <!-- <gazebo>
     <plugin name="gazebo_ros_control" filename="libgazebo_ros_control.so">
       <robotNamespace>/</robotNamespace>
     </plugin>
-  </gazebo>
+  </gazebo> -->
   <link name="world"/>
   <joint name="world_fixed" type="fixed">

File: urdf/simulation/asus_xtion.gazebo.xacro (robot description, xacro)
@@ -20,4 +20,5 @@
           </camera>
           <plugin name="${reference}_camera_controller" filename="libgazebo_ros_openni_kinect.so">
+            <robotNamespace>/</robotNamespace>
             <alwaysOn>true</alwaysOn>
             <updateRate>${update_rate}</updateRate>

File: urdf/simulation/base.gazebo.xacro (robot description, xacro)
@@ -1,11 +1,13 @@
 <?xml version="1.0"?>
 <robot xmlns:xacro="http://ros.org/wiki/xacro">
-  <xacro:macro name="gazebo_base" params="reference">
+  <xacro:macro name="gazebo_base" params="reference update_rate">
       <gazebo>
         <plugin name="${reference}_controller" filename="libgazebo_ros_planar_move.so">
+          <robotNamespace>/</robotNamespace>
           <commandTopic>cmd_vel</commandTopic>
           <odometryTopic>odom</odometryTopic>
           <odometryFrame>odom</odometryFrame>
-          <odometryRate>100.0</odometryRate>
+          <odometryRate>${update_rate}</odometryRate>
+          <cmdTimeout>-1</cmdTimeout>
           <robotBaseFrame>${reference}_footprint</robotBaseFrame>
         </plugin>

File: urdf/simulation/control.gazebo.xacro (robot description, xacro)
@@ -2,5 +2,8 @@
 <robot xmlns:xacro="http://ros.org/wiki/xacro">
   <gazebo>
-    <plugin name="gazebo_ros_control" filename="libgazebo_ros_control.so"/>
+    <plugin name="gazebo_ros_control" filename="libgazebo_ros_control.so">
+        <robotNamespace>/</robotNamespace>
+        <robotSimType>gazebo_ros_control/DefaultRobotHWSim</robotSimType>
+    </plugin>
   </gazebo>
 </robot>

File: urdf/simulation/hokuyo_urg.gazebo.xacro (robot description, xacro)
@@ -23,4 +23,5 @@
         </ray>
         <plugin name="gazebo_ros_${reference}_controller" filename="libgazebo_ros_laser.so">
+          <robotNamespace>/</robotNamespace>
           <gaussianNoise>0.005</gaussianNoise>
           <alwaysOn>true</alwaysOn>

File: urdf/simulation/hokuyo_utm.gazebo.xacro (robot description, xacro)
@@ -23,4 +23,5 @@
         </ray>
         <plugin name="gazebo_ros_${reference}_controller" filename="libgazebo_ros_laser.so">
+          <robotNamespace>/</robotNamespace>
           <gaussianNoise>0.005</gaussianNoise>
           <alwaysOn>true</alwaysOn>

File: urdf/simulation/kinect_one.gazebo.xacro (robot description, xacro)
@@ -19,4 +19,5 @@
             </camera>
             <plugin name="{reference}_camera_controller" filename="libgazebo_ros_openni_kinect.so">
+              <robotNamespace>/</robotNamespace>
               <alwaysOn>true</alwaysOn>
               <updateRate>${update_rate}</updateRate>

File: urdf/simulation/manipulator.gazebo.xacro (robot description, xacro)
@@ -84,5 +84,5 @@
     </transmission>
 <!--##################### ROS CONTROL ########################-->
-    <gazebo>
+    <!-- <gazebo>
         <plugin name="gazebo_ros_control" filename="libgazebo_ros_control.so">
         <robotNamespace></robotNamespace>
@@ -90,4 +90,5 @@
         </plugin>
     </gazebo>
+ -->
 <!--##################### GRASP FIX ########################-->
     <!-- <gazebo>
